Commit message: b

File: urdf/carpole.xacro (robot description, xacro)
@@ -4,5 +4,5 @@
   <joint name="fixed" type="fixed">
     <parent link="world"/>
-    <child link="link1"/>
+    <child link="base_rail"/>
   </joint>
   <link name="base_rail">

Commit message: linear rail added

File: urdf/carpole.xacro (robot description, xacro)
@@ -8,18 +8,18 @@
   <link name="base_rail">
     <collision>
-      <origin xyz="0 0 0" rpy="0 0 0"/>
+      <origin xyz="0 0 1.0" rpy="0 0 0"/>
       <geometry>
-        <box size="1.0 0.4 0.4"/>
+        <box size="1.0 0.04 0.04"/>
       </geometry>
     </collision>
     <visual>
-      <origin xyz="0 0 0" rpy="0 0 0"/>
+      <origin xyz="0 0 1.0" rpy="0 0 0"/>
       <geometry>
-        <box size="1.0 0.4 0.4"/>
+        <box size="1.0 0.04 0.04"/>
       </geometry>
       <material name="orange"/>
     </visual>
     <inertial>
-      <origin xyz="0 0 1" rpy="0 0 0"/>
+      <origin xyz="0.5 0.02 0.02" rpy="0 0 0"/>
       <mass value="1"/>
       <inertia

Commit message: car urdf added

File: urdf/carpole.xacro (robot description, xacro)
@@ -6,4 +6,5 @@
     <child link="base_rail"/>
   </joint>
+  <!-- rail link -->
   <link name="base_rail">
     <collision>
@@ -29,3 +30,31 @@
     </inertial>
   </link>
+  <!-- car link -->
+  <link name="car">
+    <collision>
+      <origin xyz="0 0 0" rpy="0 0 0"/>
+      <geometry>
+        <box size="0.08 0.05 0.05"/>
+      </geometry>
+    </collision>
+    <visual>
+      <origin xyz="0 0 0" rpy="0 0 0"/>
+      <geometry>
+        <box size="0.08 0.05 0.05"/>
+      </geometry>
+      <material name="orange"/>
+    </visual>
+    <inertial>
+      <origin xyz="0 0 1" rpy="0 0 0"/>
+      <mass value="1"/>
+      <inertia
+        ixx="1.0" ixy="1.0" ixz="1.0"
+        iyy="1.0" iyz="1.0"
+        izz="1.0"/>
+    </inertial>
+  </link>
+  <joint name="carsld" type="continuous">
+    <parent link="base_rail"/>
+    <child link="car"/>
+  </joint>
 </robot>

Commit message: c

File: urdf/carpole.xacro (robot description, xacro)
@@ -33,5 +33,5 @@
   <link name="car">
     <collision>
-      <origin xyz="0 0 0" rpy="0 0 0"/>
+      <origin xyz="0 0 1.02" rpy="0 0 0"/>
       <geometry>
         <box size="0.08 0.05 0.05"/>
@@ -39,5 +39,5 @@
     </collision>
     <visual>
-      <origin xyz="0 0 0" rpy="0 0 0"/>
+      <origin xyz="0 0 1.02" rpy="0 0 0"/>
       <geometry>
         <box size="0.08 0.05 0.05"/>

Commit message: linear rail joint added

File: urdf/carpole.xacro (robot description, xacro)
@@ -34,18 +34,18 @@
   <link name="car">
     <collision>
-      <origin xyz="0 0 1.02" rpy="0 0 0"/>
+      <origin xyz="0 0 1.045" rpy="0 0 0"/>
       <geometry>
-        <box size="0.08 0.05 0.05"/>
+        <box size="0.08 0.08 0.05"/>
       </geometry>
     </collision>
     <visual>
-      <origin xyz="0 0 1.02" rpy="0 0 0"/>
+      <origin xyz="0 0 1.045" rpy="0 0 0"/>
       <geometry>
-        <box size="0.08 0.05 0.05"/>
+        <box size="0.08 0.08 0.05"/>
       </geometry>
       <material name="orange"/>
     </visual>
     <inertial>
-      <origin xyz="0 0 1" rpy="0 0 0"/>
+      <origin xyz="0 0 1.045" rpy="0 0 0"/>
       <mass value="1"/>
       <inertia
@@ -55,7 +55,12 @@
     </inertial>
   </link>
-  <joint name="carsld" type="continuous">
+  <joint name="carsld" type="prismatic">
     <parent link="base_rail"/>
     <child link="car"/>
+    <axis xyz="1 0 0"/>
+    <limit lower="-0.4"
+         upper="0.4"
+         effort="10.0"
+         velocity="1005.0" />
   </joint>
 </robot>

Commit message: car-pole model done(URDF)

File: urdf/carpole.xacro (robot description, xacro)
@@ -64,3 +64,38 @@
          velocity="1005.0" />
   </joint>
+  <!-- pendu link -->
+  <link name="bar">
+    <collision>
+      <origin xyz="0.3 -0.005 0" rpy="0 0 0"/>
+      <geometry>
+        <box size="0.6 0.01 0.01"/>
+      </geometry>
+    </collision>
+    <visual>
+      <origin xyz="0.3 -0.005 0" rpy="0 0 0"/>
+      <geometry>
+        <box size="0.6 0.01 0.01"/>
+      </geometry>
+      <material name="orange"/>
+    </visual>
+    <inertial>
+      <origin xyz="0.6 -0.005 0.005" rpy="0 0 0"/>
+      <mass value="2.1"/>
+      <inertia
+        ixx="1.0" ixy="1.0" ixz="1.0"
+        iyy="1.0" iyz="1.0"
+        izz="1.0"/>
+    </inertial>
+  </link>
+  <joint name="bar_car" type="continuous">
+    <parent link="car"/>
+    <child link="bar"/>
+    <origin xyz="0.0 -0.04 1.045" rpy="0 0 0"/>
+    <axis xyz="0 1 0" rpy="0 0 0"/>
+    <limit effort="10.0" velocity="1005.0" />
+  </joint>
+  <!-- <joint name="bar_car" type="fixed">
+    <parent link="world"/>
+    <child link="bar"/>
+  </joint> -->
 </robot>

Commit message: model done

File: urdf/carpole.xacro (robot description, xacro)
@@ -99,3 +99,32 @@
     <child link="bar"/>
   </joint> -->
+  <!-- end mass -->
+  <link name="mass">
+    <collision>
+      <origin xyz="0 0 0" rpy="0 0 `0"/>
+      <geometry>
+        <box size="0.05 0.05 0.05"/>
+      </geometry>
+    </collision>
+    <visual>
+      <origin xyz="0 0 0" rpy="0 0 0"/>
+      <geometry>
+        <box size="0.05 0.05 0.05"/>
+      </geometry>
+      <material name="orange"/>
+    </visual>
+    <inertial>
+      <origin xyz="0 0 0" rpy="0 0 0"/>
+      <mass value="1"/>
+      <inertia
+        ixx="0.0004089" ixy="0" ixz="0"
+        iyy="0.0004089" iyz="0"
+        izz="0.0004089"/>
+    </inertial>
+  </link>
+  <joint name="bar_mass" type="fixed">
+    <parent link="bar"/>
+    <child link="mass"/>
+    <origin xyz="0.575 -0.005 0" rpy="0 0 0"/>
+  </joint>
 </robot>

Commit message: joint controller added and configed

File: urdf/carpole.xacro (robot description, xacro)
@@ -61,5 +61,5 @@
     <limit lower="-0.4"
          upper="0.4"
-         effort="10.0"
+         effort="1000.0"
          velocity="1005.0" />
   </joint>
@@ -81,9 +81,9 @@
     <inertial>
       <origin xyz="0.6 -0.005 0.005" rpy="0 0 0"/>
-      <mass value="2.1"/>
+      <mass value="0.000001"/>
       <inertia
-        ixx="1.0" ixy="1.0" ixz="1.0"
-        iyy="1.0" iyz="1.0"
-        izz="1.0"/>
+        ixx="0.000001" ixy="0.0" ixz="0.0"
+        iyy="0.000001" iyz="0.0"
+        izz="0.000001"/>
     </inertial>
   </link>
@@ -93,5 +93,5 @@
     <origin xyz="0.0 -0.04 1.045" rpy="0 0 0"/>
     <axis xyz="0 1 0" rpy="0 0 0"/>
-    <limit effort="10.0" velocity="1005.0" />
+    <limit effort="1000.0" velocity="1005.0" />
   </joint>
   <!-- <joint name="bar_car" type="fixed">
@@ -102,5 +102,5 @@
   <link name="mass">
     <collision>
-      <origin xyz="0 0 0" rpy="0 0 `0"/>
+      <origin xyz="0 0 0" rpy="0 0 0"/>
       <geometry>
         <box size="0.05 0.05 0.05"/>
@@ -118,7 +118,7 @@
       <mass value="1"/>
       <inertia
-        ixx="0.0004089" ixy="0" ixz="0"
-        iyy="0.0004089" iyz="0"
-        izz="0.0004089"/>
+        ixx="0.0004" ixy="0" ixz="0"
+        iyy="0.0004" iyz="0"
+        izz="0.0004"/>
     </inertial>
   </link>
@@ -128,3 +128,14 @@
     <origin xyz="0.575 -0.005 0" rpy="0 0 0"/>
   </joint>
+  <!-- transmission for the car on the linear rail  -->
+  <transmission name="linear_rail">
+    <type>transmission_interface/SimpleTransmission</type>
+    <joint name="carsld">
+      <hardwareInterface>hardware_interface/EffortJointInterface</hardwareInterface>
+    </joint>
+    <actuator name="motor1">
+      <hardwareInterface>hardware_interface/EffortJointInterface</hardwareInterface>
+      <mechanicalReduction>1</mechanicalReduction>
+    </actuator>
+  </transmission>
 </robot>

Commit message: energy forming code added

File: urdf/carpole.xacro (robot description, xacro)
@@ -3,36 +3,30 @@
   <xacro:include filename="$(find carpole)/urdf/carpole.gazebo" />
   <link name="world"/>
-  <joint name="fixed" type="fixed">
-    <parent link="world"/>
-    <child link="base_rail"/>
-  </joint>
-  <!-- rail link -->
   <link name="base_rail">
     <collision>
-      <origin xyz="0 0 1.0" rpy="0 0 0"/>
+      <origin xyz="0 0 0" rpy="0 0 0"/>
       <geometry>
-        <box size="1.0 0.04 0.04"/>
+        <box size="2.0 0.04 0.04"/>
       </geometry>
     </collision>
     <visual>
-      <origin xyz="0 0 1.0" rpy="0 0 0"/>
+      <origin xyz="0 0 0" rpy="0 0 0"/>
       <geometry>
-        <box size="1.0 0.04 0.04"/>
+        <box size="2.0 0.04 0.04"/>
       </geometry>
       <material name="orange"/>
     </visual>
     <inertial>
-      <origin xyz="0.5 0.02 0.02" rpy="0 0 0"/>
+      <origin xyz="0 0 0" rpy="0 0 0"/>
       <mass value="1"/>
       <inertia
-        ixx="1.0" ixy="1.0" ixz="1.0"
-        iyy="1.0" iyz="1.0"
+        ixx="1.0" ixy="0.0" ixz="0.0"
+        iyy="1.0" iyz="0.0"
         izz="1.0"/>
     </inertial>
   </link>
-  <!-- car link -->
   <link name="car">
     <collision>
-      <origin xyz="0 0 1.045" rpy="0 0 0"/>
+      <origin xyz="0 0 0" rpy="0 0 0"/>
       <geometry>
         <box size="0.08 0.08 0.05"/>
@@ -40,29 +34,18 @@
     </collision>
     <visual>
-      <origin xyz="0 0 1.045" rpy="0 0 0"/>
+      <origin xyz="0 0 0" rpy="0 0 0"/>
       <geometry>
         <box size="0.08 0.08 0.05"/>
       </geometry>
-      <material name="orange"/>
     </visual>
     <inertial>
-      <origin xyz="0 0 1.045" rpy="0 0 0"/>
-      <mass value="1"/>
+      <origin xyz="0 0 0" rpy="0 0 0"/>
+      <mass value="1.0"/>
       <inertia
-        ixx="1.0" ixy="1.0" ixz="1.0"
-        iyy="1.0" iyz="1.0"
-        izz="1.0"/>
+        ixx="0.1" ixy="0.0" ixz="0.0"
+        iyy="0.1" iyz="0.0"
+        izz="0.1"/>
     </inertial>
   </link>
-  <joint name="carsld" type="prismatic">
-    <parent link="base_rail"/>
-    <child link="car"/>
-    <axis xyz="1 0 0"/>
-    <limit lower="-0.4"
-         upper="0.4"
-         effort="1000.0"
-         velocity="1005.0" />
-  </joint>
-  <!-- pendu link -->
   <link name="bar">
     <collision>
@@ -77,32 +60,19 @@
         <box size="0.6 0.01 0.01"/>
       </geometry>
-      <material name="orange"/>
     </visual>
     <inertial>
-      <origin xyz="0.6 -0.005 0.005" rpy="0 0 0"/>
-      <mass value="0.000001"/>
+      <origin xyz="0.3 -0.005 0" rpy="0 0 0"/>
+      <mass value="0.001"/>
       <inertia
-        ixx="0.000001" ixy="0.0" ixz="0.0"
-        iyy="0.000001" iyz="0.0"
-        izz="0.000001"/>
+        ixx="0.001" ixy="0.0" ixz="0.0"
+        iyy="0.001" iyz="0.0"
+        izz="0.001"/>
     </inertial>
   </link>
-  <joint name="bar_car" type="continuous">
-    <parent link="car"/>
-    <child link="bar"/>
-    <origin xyz="0.0 -0.04 1.045" rpy="0 0 0"/>
-    <axis xyz="0 1 0" rpy="0 0 0"/>
-    <limit effort="1000.0" velocity="1005.0" />
-  </joint>
-  <!-- <joint name="bar_car" type="fixed">
-    <parent link="world"/>
-    <child link="bar"/>
-  </joint> -->
-  <!-- end mass -->
-  <link name="mass">
+  <link name="masspoint">
     <collision>
       <origin xyz="0 0 0" rpy="0 0 0"/>
       <geometry>
-        <box size="0.05 0.05 0.05"/>
+        <box size="0.02 0.02 0.02"/>
       </geometry>
     </collision>
@@ -110,23 +80,44 @@
       <origin xyz="0 0 0" rpy="0 0 0"/>
       <geometry>
-        <box size="0.05 0.05 0.05"/>
+        <box size="0.02 0.02 0.02"/>
       </geometry>
-      <material name="orange"/>
     </visual>
     <inertial>
       <origin xyz="0 0 0" rpy="0 0 0"/>
-      <mass value="1"/>
+      <mass value="3.0"/>
       <inertia
-        ixx="0.0004" ixy="0" ixz="0"
-        iyy="0.0004" iyz="0"
-        izz="0.0004"/>
+        ixx="0.1" ixy="0" ixz="0"
+        iyy="0.1" iyz="0"
+        izz="0.1"/>
     </inertial>
   </link>
+  <joint name="fixedjoint" type="fixed">
+    <parent link="world"/>
+    <child link="base_rail"/>
+    <origin xyz="0 0 1" rpy="0 0 0"/>
+  </joint>
+  <joint name="carsld" type="prismatic">
+    <parent link="base_rail"/>
+    <child link="car"/>
+    <origin xyz="0 0 0.045" rpy="0 0 0"/>
+    <axis xyz="1 0 0"/>
+    <limit lower="-1"
+         upper="1"
+         effort="1000.0"
+         velocity="1005.0" />
+  </joint>
+  <joint name="bar_car" type="continuous">
+    <parent link="car"/>
+    <child link="bar"/>
+    <origin xyz="0 -0.04 0" rpy="0 0 0"/>
+    <axis xyz="0 1 0"/>
+    <!-- <hardwareInterface>hardware_interface/EffortJointInterface</hardwareInterface> -->
+    <!-- <anchor xyz="0 0 0"/> -->
+  </joint>
   <joint name="bar_mass" type="fixed">
     <parent link="bar"/>
-    <child link="mass"/>
-    <origin xyz="0.575 -0.005 0" rpy="0 0 0"/>
+    <child link="masspoint"/>
+    <origin xyz="0.6 -0.005 0" rpy="0 0 0"/>
   </joint>
-  <!-- transmission for the car on the linear rail  -->
   <transmission name="linear_rail">
     <type>transmission_interface/SimpleTransmission</type>
@@ -139,3 +130,13 @@
     </actuator>
   </transmission>
+  <transmission name="bar_car">
+    <type>transmission_interface/SimpleTransmission</type>
+    <joint name="bar_car">
+      <hardwareInterface>hardware_interface/EffortJointInterface</hardwareInterface>
+    </joint>
+    <actuator name="motor2">
+      <hardwareInterface>hardware_interface/EffortJointInterface</hardwareInterface>
+      <mechanicalReduction>1</mechanicalReduction>
+    </actuator>
+  </transmission>
 </robot>

Commit message: energy shaping control parameters tuned

File: urdf/carpole.xacro (robot description, xacro)
@@ -106,4 +106,5 @@
          effort="1000.0"
          velocity="1005.0" />
+    <dynamics damping="0.5" friction="0.3"/>
   </joint>
   <joint name="bar_car" type="continuous">

Commit message: swing up energy modified

File: urdf/carpole.xacro (robot description, xacro)
@@ -85,5 +85,5 @@
     <inertial>
       <origin xyz="0 0 0" rpy="0 0 0"/>
-      <mass value="3.0"/>
+      <mass value="2.0"/>
       <inertia
         ixx="0.1" ixy="0" ixz="0"
@@ -102,9 +102,9 @@
     <origin xyz="0 0 0.045" rpy="0 0 0"/>
     <axis xyz="1 0 0"/>
-    <limit lower="-1"
-         upper="1"
-         effort="1000.0"
-         velocity="1005.0" />
-    <dynamics damping="0.5" friction="0.3"/>
+    <limit lower="-1.5"
+         upper="1.5"
+         effort="100000.0"
+         velocity="100005.0" />
+    <dynamics damping="0.0" friction="0.0"/>
   </joint>
   <joint name="bar_car" type="continuous">

Commit message: setup on cube case

File: urdf/carpole.xacro (robot description, xacro)
@@ -102,6 +102,6 @@
     <origin xyz="0 0 0.045" rpy="0 0 0"/>
     <axis xyz="1 0 0"/>
-    <limit lower="-1.5"
-         upper="1.5"
+    <limit lower="-1.0"
+         upper="1.0"
          effort="100000.0"
          velocity="100005.0" />
